File: designs/3.3V Step Down Converter/untitled.sch (EAGLE design)
At the start: 10 parts, among them IC1 TPS62160DGKR, J1 S2B-PH-SM4, J2 S2B-PH-SM4

Commit message: inductor change
Parts:
- L1: value 2.2uH -> VLS6045EX-221M; device MouserUseful:VLS6045EX-1R5N -> MouserUseful:VLS6045EX-221M
Changed lines of the file:
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@@
 <?xml version="1.0" encoding="utf-8"?>
 <!DOCTYPE eagle SYSTEM "eagle.dtd">
-<eagle version="9.4.2">
+<eagle version="9.5.1">
 <drawing>
 <settings>
@@
 <part name="R1" library="MouserUseful" deviceset="RCS1206100KJNEA" device="R1206" package3d_urn="urn:adsk.eagle:package:23540/2" value="100kOhm"/>
 <part name="R3" library="MouserUseful" deviceset="RN73R1ETTP1803D25" device="R0402" package3d_urn="urn:adsk.eagle:package:26058/2" value="180kOhm"/>
-<part name="L1" library="MouserUseful" deviceset="VLS6045EX-1R5N" device="" package3d_urn="urn:adsk.eagle:package:13422172/1" value="2.2uH"/>
 <part name="AGND1" library="supply1" library_urn="urn:adsk.eagle:library:371" deviceset="AGND" device=""/>
 <part name="JP1" library="pinhead" library_urn="urn:adsk.eagle:library:325" deviceset="PINHD-1X4" device="" package3d_urn="urn:adsk.eagle:package:22407/2"/>
@@
 <part name="AGND2" library="supply1" library_urn="urn:adsk.eagle:library:371" deviceset="AGND" device=""/>
 <part name="AGND3" library="supply1" library_urn="urn:adsk.eagle:library:371" deviceset="AGND" device=""/>
+<part name="L1" library="MouserUseful" deviceset="VLS6045EX-221M" device=""/>
 </parts>
 <sheets>
@@
 <attribute name="VALUE" x="137.922" y="125.73" size="1.778" layer="96" rot="R90"/>
 </instance>
+<instance part="AGND1" gate="VR1" x="81.28" y="114.3" smashed="yes">
+<attribute name="VALUE" x="78.74" y="109.22" size="1.778" layer="96" rot="R90"/>
+</instance>
+<instance part="JP1" gate="A" x="142.24" y="114.3" smashed="yes" rot="R90">
+<attribute name="NAME" x="133.985" y="107.95" size="1.778" layer="95" rot="R90"/>
+<attribute name="VALUE" x="149.86" y="107.95" size="1.778" layer="96" rot="R90"/>
+</instance>
+<instance part="AGND4" gate="VR1" x="139.7" y="93.98" smashed="yes">
+<attribute name="VALUE" x="137.16" y="88.9" size="1.778" layer="96" rot="R90"/>
+</instance>
+<instance part="AGND5" gate="VR1" x="142.24" y="93.98" smashed="yes">
+<attribute name="VALUE" x="139.7" y="88.9" size="1.778" layer="96" rot="R90"/>
+</instance>
+<instance part="J1" gate="G$1" x="104.14" y="111.76" smashed="yes" rot="R90">
+<attribute name="NAME" x="98.54428125" y="106.6771" size="1.272509375" layer="95" rot="R90"/>
+<attribute name="VALUE" x="113.56268125" y="106.67188125" size="1.275409375" layer="96" rot="R90"/>
+</instance>
+<instance part="J2" gate="G$1" x="121.92" y="111.76" smashed="yes" rot="R90">
+<attribute name="NAME" x="116.32428125" y="106.6771" size="1.272509375" layer="95" rot="R90"/>
+<attribute name="VALUE" x="131.34268125" y="106.67188125" size="1.275409375" layer="96" rot="R90"/>
+</instance>
+<instance part="AGND2" gate="VR1" x="109.22" y="91.44" smashed="yes">
+<attribute name="VALUE" x="106.68" y="86.36" size="1.778" layer="96" rot="R90"/>
+</instance>
+<instance part="AGND3" gate="VR1" x="127" y="91.44" smashed="yes">
+<attribute name="VALUE" x="124.46" y="86.36" size="1.778" layer="96" rot="R90"/>
+</instance>
 <instance part="L1" gate="G$1" x="106.68" y="154.94" smashed="yes">
 <attribute name="NAME" x="123.19" y="161.29" size="1.778" layer="95" align="center-left"/>
 <attribute name="VALUE" x="123.19" y="158.75" size="1.778" layer="96" align="center-left"/>
-</instance>
-<instance part="AGND1" gate="VR1" x="81.28" y="114.3" smashed="yes">
-<attribute name="VALUE" x="78.74" y="109.22" size="1.778" layer="96" rot="R90"/>
-</instance>
-<instance part="JP1" gate="A" x="142.24" y="114.3" smashed="yes" rot="R90">
-<attribute name="NAME" x="133.985" y="107.95" size="1.778" layer="95" rot="R90"/>
-<attribute name="VALUE" x="149.86" y="107.95" size="1.778" layer="96" rot="R90"/>
-</instance>
-<instance part="AGND4" gate="VR1" x="139.7" y="93.98" smashed="yes">
-<attribute name="VALUE" x="137.16" y="88.9" size="1.778" layer="96" rot="R90"/>
-</instance>
-<instance part="AGND5" gate="VR1" x="142.24" y="93.98" smashed="yes">
-<attribute name="VALUE" x="139.7" y="88.9" size="1.778" layer="96" rot="R90"/>
-</instance>
-<instance part="J1" gate="G$1" x="104.14" y="111.76" smashed="yes" rot="R90">
-<attribute name="NAME" x="98.54428125" y="106.6771" size="1.272509375" layer="95" rot="R90"/>
-<attribute name="VALUE" x="113.56268125" y="106.67188125" size="1.275409375" layer="96" rot="R90"/>
-</instance>
-<instance part="J2" gate="G$1" x="121.92" y="111.76" smashed="yes" rot="R90">
-<attribute name="NAME" x="116.32428125" y="106.6771" size="1.272509375" layer="95" rot="R90"/>
-<attribute name="VALUE" x="131.34268125" y="106.67188125" size="1.275409375" layer="96" rot="R90"/>
-</instance>
-<instance part="AGND2" gate="VR1" x="109.22" y="91.44" smashed="yes">
-<attribute name="VALUE" x="106.68" y="86.36" size="1.778" layer="96" rot="R90"/>
-</instance>
-<instance part="AGND3" gate="VR1" x="127" y="91.44" smashed="yes">
-<attribute name="VALUE" x="124.46" y="86.36" size="1.778" layer="96" rot="R90"/>
 </instance>
 </instances>
@@
 <pinref part="R1" gate="G$1" pin="2"/>
 <wire x1="121.92" y1="144.78" x2="127" y2="144.78" width="0.1524" layer="91"/>
-<pinref part="L1" gate="G$1" pin="2"/>
 <wire x1="127" y1="154.94" x2="134.62" y2="154.94" width="0.1524" layer="91"/>
 <wire x1="134.62" y1="154.94" x2="147.32" y2="154.94" width="0.1524" layer="91"/>
@@
 <wire x1="127" y1="144.78" x2="127" y2="154.94" width="0.1524" layer="91"/>
 <junction x="127" y="144.78"/>
-<junction x="127" y="154.94"/>
 <pinref part="R2" gate="G$1" pin="2"/>
 <wire x1="134.62" y1="149.86" x2="134.62" y2="154.94" width="0.1524" layer="91"/>
@@
 <junction x="147.32" y="154.94"/>
 <label x="152.4" y="154.94" size="1.778" layer="95" xref="yes"/>
+<pinref part="L1" gate="G$1" pin="2"/>
+<junction x="127" y="154.94"/>
 </segment>
 <segment>
@@
 <pinref part="IC1" gate="G$1" pin="SW"/>
 <wire x1="104.14" y1="142.24" x2="106.68" y2="142.24" width="0.1524" layer="91"/>
+<wire x1="106.68" y1="142.24" x2="106.68" y2="154.94" width="0.1524" layer="91"/>
 <pinref part="L1" gate="G$1" pin="1"/>
-<wire x1="106.68" y1="142.24" x2="106.68" y2="154.94" width="0.1524" layer="91"/>
-</segment>
-</net>
+</segment>
+</net>
