File: designs/MainBoard/MainBoard.sch (EAGLE design)
At the start: 6 parts

Commit message: finished mainboard
Parts:
- removed SV1: (no value), con-lstb:MA08-1
- added J1, J2, J3, J4, J5, J6, J7, J8: S2B-PH-SM4, CommonParts:S2B-PH-SM4
- added R1, R2, R3, R4: (no value), CommonParts:R-EU_1206R1206
- added SV4: (no value), CommonParts:PINHEADER-1X8
Connections:
- net 3.3V: now also J2.1, J4.1, J6.1, J8.1, R1.1, R2.1, R3.1, R4.1, SV4.7; no longer SV1.7
- net GND: now also J1.2, J2.2, J3.2, J4.2, J5.2, J6.2, J7.2, J8.2, SV4.8; no longer SV1.8
- net GPIO13: now also SV4.4; no longer SV1.4
- net IO15: now also J1.1, R1.2
- net IO2: now also SV4.3; no longer SV1.3
- net IO22: now also J7.1, R4.2
- net IO25: now also SV4.5; no longer SV1.5
- net IO26: now also SV4.6; no longer SV1.6
- net IO4: now also SV4.1; no longer SV1.1
- net IO5: now also SV4.2; no longer SV1.2
- net RXD0: now also J3.1, R2.2
- net TXD0: now also J5.1, R3.2

Commit message: added last design tunes
Parts:
- R1, R2, R3, R4: value (none) -> 10K
Changed lines of the file:
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@@
 <part name="J7" library="CommonParts" deviceset="S2B-PH-SM4" device=""/>
 <part name="J8" library="CommonParts" deviceset="S2B-PH-SM4" device=""/>
-<part name="R1" library="CommonParts" deviceset="R-EU_1206" device="R1206" package3d_urn="urn:adsk.eagle:package:23540/2"/>
-<part name="R2" library="CommonParts" deviceset="R-EU_1206" device="R1206" package3d_urn="urn:adsk.eagle:package:23540/2"/>
-<part name="R3" library="CommonParts" deviceset="R-EU_1206" device="R1206" package3d_urn="urn:adsk.eagle:package:23540/2"/>
-<part name="R4" library="CommonParts" deviceset="R-EU_1206" device="R1206" package3d_urn="urn:adsk.eagle:package:23540/2"/>
+<part name="R1" library="CommonParts" deviceset="R-EU_1206" device="R1206" package3d_urn="urn:adsk.eagle:package:23540/2" value="10K"/>
+<part name="R2" library="CommonParts" deviceset="R-EU_1206" device="R1206" package3d_urn="urn:adsk.eagle:package:23540/2" value="10K"/>
+<part name="R3" library="CommonParts" deviceset="R-EU_1206" device="R1206" package3d_urn="urn:adsk.eagle:package:23540/2" value="10K"/>
+<part name="R4" library="CommonParts" deviceset="R-EU_1206" device="R1206" package3d_urn="urn:adsk.eagle:package:23540/2" value="10K"/>
 <part name="SV4" library="CommonParts" deviceset="PINHEADER-1X8" device="" package3d_urn="urn:adsk.eagle:package:8343/1"/>
 <part name="GND3" library="supply1" library_urn="urn:adsk.eagle:library:371" deviceset="GND" device=""/>
