File: designs/ESP32WroverB/untitled.sch (EAGLE design)
At the start: 19 parts, among them IC6 ESP32-WROVER-B

Commit message: added design block Logo
Parts:
- removed BOOT: (no value), CommonParts:PINHEADER-1X2
- removed SV3, SV4: (no value), con-lstb:MA09-1
- added RST: FSMSMTR, FSMSMTR:FSMSMTR
- added SV5, SV6: (no value), CommonParts:PINHEADER-1X9
- SV1, SV2: device con-lstb:MA09-1 -> CommonParts:PINHEADER-1X9
- renumbered ENABLE to EN
Connections:
- net 3.3V: now also SV5.8; no longer ON/OFF.3, SV1.8
- net CLK: now also SV1.9; no longer SV3.9
- net CMD: now also SV6.1; no longer SV2.1
- net EN: now also SV5.7; no longer SV1.7
- net GND: now also RST.2, SV5.9; no longer BOOT.2, SV1.9
- net GPIO12: now also SV6.5; no longer SV2.5
- net GPIO13: now also SV6.4; no longer SV2.4
- net GPIO14: now also SV6.6; no longer SV2.6
- net IO0: now also RST.1, SV1.4; no longer BOOT.1, SV3.4
- net IO15: now also SV1.6; no longer SV3.6
- net IO18: now also SV2.8; no longer SV4.8
- net IO19: now also SV2.7; no longer SV4.7
- net IO2: now also SV1.5; no longer SV3.5
- net IO21: now also SV2.5; no longer SV4.5
- net IO22: now also SV2.2; no longer SV4.2
- net IO23: now also SV2.1; no longer SV4.1
- net IO25: now also SV6.9; no longer SV2.9
- net IO26: now also SV6.8; no longer SV2.8
- net IO27: now also SV6.7; no longer SV2.7
- net IO32: now also SV5.2; no longer SV1.2
- net IO33: now also SV5.1; no longer SV1.1
- net IO34: now also SV5.4; no longer SV1.4
- net IO35: now also SV5.3; no longer SV1.3
- net IO4: now also SV1.3; no longer SV3.3
- net IO5: now also SV2.9; no longer SV4.9
- net NC_1: now also SV1.2; no longer SV3.2
- net NC_2: now also SV1.1; no longer SV3.1
- net NC_3: now also SV2.6; no longer SV4.6
- net RXD0: now also SV2.4; no longer SV4.4
- net SD0: now also SV1.8; no longer SV3.8
- net SD1: now also SV1.7; no longer SV3.7
- net SD2: now also SV6.3; no longer SV2.3
- net SD3: now also SV6.2; no longer SV2.2
- net SEN_VN: now also SV5.5; no longer SV1.5
- net SEN_VP: now also SV5.6; no longer SV1.6
- net TXD0: now also SV2.3; no longer SV4.3

Commit message: added last design tunes
Changed lines of the file:
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@@
 <?xml version="1.0" encoding="utf-8"?>
 <!DOCTYPE eagle SYSTEM "eagle.dtd">
-<eagle version="9.4.2">
+<eagle version="9.5.1">
 <drawing>
 <settings>
@@
 <pinref part="IC6" gate="G$1" pin="GND_3"/>
 <wire x1="160.02" y1="162.56" x2="167.64" y2="162.56" width="0.1524" layer="91"/>
-<wire x1="167.64" y1="162.56" x2="167.64" y2="160.02" width="0.1524" layer="91"/>
-<pinref part="IC6" gate="G$1" pin="GND_4"/>
 <wire x1="167.64" y1="149.86" x2="167.64" y2="154.94" width="0.1524" layer="91"/>
 <wire x1="167.64" y1="154.94" x2="167.64" y2="160.02" width="0.1524" layer="91"/>
-<wire x1="167.64" y1="160.02" x2="160.02" y2="160.02" width="0.1524" layer="91"/>
 <pinref part="GND15" gate="1" pin="GND"/>
+<wire x1="167.64" y1="160.02" x2="167.64" y2="162.56" width="0.1524" layer="91"/>
 <wire x1="172.72" y1="154.94" x2="167.64" y2="154.94" width="0.1524" layer="91"/>
 <junction x="167.64" y="154.94"/>
 <pinref part="RST" gate="G$1" pin="2"/>
 <wire x1="172.72" y1="167.64" x2="172.72" y2="154.94" width="0.1524" layer="91"/>
+<pinref part="IC6" gate="G$1" pin="GND_4"/>
+<wire x1="160.02" y1="160.02" x2="167.64" y2="160.02" width="0.1524" layer="91"/>
+<junction x="167.64" y="160.02"/>
 </segment>
 <segment>
@@
 </sheet>
 </sheets>
+<errors>
+</errors>
 </schematic>
 </drawing>

Commit message: added ESP32 Capacitor values
Parts:
- C1, C4: value (none) -> 1nF
- C2: value (none) -> 100uF
- C3: value (none) -> 1uF
Changed lines of the file:
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@@
 <part name="GND20" library="supply1" library_urn="urn:adsk.eagle:library:371" deviceset="GND" device=""/>
 <part name="GND13" library="supply1" library_urn="urn:adsk.eagle:library:371" deviceset="GND" device=""/>
-<part name="C1" library="CommonParts" deviceset="C-EU_805" device="C0805" package3d_urn="urn:adsk.eagle:package:23617/2"/>
-<part name="C2" library="CommonParts" deviceset="C-EU_805" device="C0805" package3d_urn="urn:adsk.eagle:package:23617/2"/>
-<part name="C3" library="CommonParts" deviceset="C-EU_805" device="C0805" package3d_urn="urn:adsk.eagle:package:23617/2"/>
+<part name="C1" library="CommonParts" deviceset="C-EU_805" device="C0805" package3d_urn="urn:adsk.eagle:package:23617/2" value="1nF"/>
+<part name="C2" library="CommonParts" deviceset="C-EU_805" device="C0805" package3d_urn="urn:adsk.eagle:package:23617/2" value="100uF"/>
+<part name="C3" library="CommonParts" deviceset="C-EU_805" device="C0805" package3d_urn="urn:adsk.eagle:package:23617/2" value="1uF"/>
 <part name="R1" library="CommonParts" deviceset="R-EU_805" device="R0805" package3d_urn="urn:adsk.eagle:package:23553/2" value="10k"/>
-<part name="C4" library="CommonParts" deviceset="C-EU_805" device="C0805" package3d_urn="urn:adsk.eagle:package:23617/2"/>
+<part name="C4" library="CommonParts" deviceset="C-EU_805" device="C0805" package3d_urn="urn:adsk.eagle:package:23617/2" value="1nF"/>
 <part name="GND1" library="supply1" library_urn="urn:adsk.eagle:library:371" deviceset="GND" device=""/>
 <part name="GND2" library="supply1" library_urn="urn:adsk.eagle:library:371" deviceset="GND" device=""/>

Commit message: corrected ESP32 on/off error
Parts:
- R1: value 10k -> 12k
- R2: value (none) -> 460ohm
Connections:
- new net N$1: ON/OFF.2, POWER.2
- net 3.3V: no longer ON/OFF.2, POWER.2
Changed lines of the file:
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@@
 <part name="C2" library="CommonParts" deviceset="C-EU_805" device="C0805" package3d_urn="urn:adsk.eagle:package:23617/2" value="100uF"/>
 <part name="C3" library="CommonParts" deviceset="C-EU_805" device="C0805" package3d_urn="urn:adsk.eagle:package:23617/2" value="1uF"/>
-<part name="R1" library="CommonParts" deviceset="R-EU_805" device="R0805" package3d_urn="urn:adsk.eagle:package:23553/2" value="10k"/>
+<part name="R1" library="CommonParts" deviceset="R-EU_805" device="R0805" package3d_urn="urn:adsk.eagle:package:23553/2" value="12k"/>
 <part name="C4" library="CommonParts" deviceset="C-EU_805" device="C0805" package3d_urn="urn:adsk.eagle:package:23617/2" value="1nF"/>
 <part name="GND1" library="supply1" library_urn="urn:adsk.eagle:library:371" deviceset="GND" device=""/>
 <part name="GND2" library="supply1" library_urn="urn:adsk.eagle:library:371" deviceset="GND" device=""/>
-<part name="R2" library="CommonParts" deviceset="R-EU_805" device="R0805" package3d_urn="urn:adsk.eagle:package:23553/2"/>
+<part name="R2" library="CommonParts" deviceset="R-EU_805" device="R0805" package3d_urn="urn:adsk.eagle:package:23553/2" value="460ohm"/>
 <part name="JTAG" library="con-lstb" library_urn="urn:adsk.eagle:library:162" deviceset="MA04-1" device="" package3d_urn="urn:adsk.eagle:package:8337/1" value="1"/>
 <part name="UART" library="con-panduit" library_urn="urn:adsk.eagle:library:169" deviceset="057-006-" device="1" package3d_urn="urn:adsk.eagle:package:9198/1"/>
@@
 </segment>
 <segment>
-<pinref part="POWER" gate="G$1" pin="2"/>
-<pinref part="ON/OFF" gate="G$1" pin="2"/>
-<wire x1="96.52" y1="247.65" x2="107.95" y2="247.65" width="0.1524" layer="91"/>
-<wire x1="107.95" y1="247.65" x2="107.95" y2="250.19" width="0.1524" layer="91"/>
-</segment>
-<segment>
 <wire x1="215.9" y1="208.28" x2="226.06" y2="208.28" width="0.1524" layer="91"/>
 <label x="215.9" y="208.28" size="1.778" layer="95"/>
@@
 </segment>
 </net>
+<net name="N$1" class="0">
+<segment>
+<pinref part="POWER" gate="G$1" pin="2"/>
+<pinref part="ON/OFF" gate="G$1" pin="2"/>
+<wire x1="96.52" y1="247.65" x2="107.95" y2="247.65" width="0.1524" layer="91"/>
+<wire x1="107.95" y1="247.65" x2="107.95" y2="250.19" width="0.1524" layer="91"/>
+</segment>
+</net>

Commit message: changed 1206 100uF Capacitor
Parts:
- C2: device CommonParts:C-EU_805C0805 -> CommonParts:C-EU_1206C1206
Changed lines of the file:
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@@
 <?xml version="1.0" encoding="utf-8"?>
 <!DOCTYPE eagle SYSTEM "eagle.dtd">
-<eagle version="9.5.1">
+<eagle version="9.4.2">
 <drawing>
 <settings>
@@
 <part name="GND13" library="supply1" library_urn="urn:adsk.eagle:library:371" deviceset="GND" device=""/>
 <part name="C1" library="CommonParts" deviceset="C-EU_805" device="C0805" package3d_urn="urn:adsk.eagle:package:23617/2" value="1nF"/>
-<part name="C2" library="CommonParts" deviceset="C-EU_805" device="C0805" package3d_urn="urn:adsk.eagle:package:23617/2" value="100uF"/>
 <part name="C3" library="CommonParts" deviceset="C-EU_805" device="C0805" package3d_urn="urn:adsk.eagle:package:23617/2" value="1uF"/>
 <part name="R1" library="CommonParts" deviceset="R-EU_805" device="R0805" package3d_urn="urn:adsk.eagle:package:23553/2" value="12k"/>
@@
 <part name="SV2" library="CommonParts" deviceset="PINHEADER-1X9" device="" package3d_urn="urn:adsk.eagle:package:8350/1"/>
 <part name="RST" library="FSMSMTR" deviceset="FSMSMTR" device=""/>
+<part name="C2" library="CommonParts" deviceset="C-EU_1206" device="C1206" package3d_urn="urn:adsk.eagle:package:23618/2" value="100uF"/>
 </parts>
 <sheets>
@@
 <attribute name="VALUE" x="217.043" y="248.666" size="1.778" layer="96" rot="R270"/>
 </instance>
-<instance part="C2" gate="G$1" x="88.9" y="198.12" smashed="yes">
-<attribute name="NAME" x="90.424" y="198.501" size="1.778" layer="95"/>
-<attribute name="VALUE" x="90.424" y="193.421" size="1.778" layer="96"/>
-</instance>
 <instance part="C3" gate="G$1" x="101.6" y="198.12" smashed="yes">
 <attribute name="NAME" x="103.124" y="198.501" size="1.778" layer="95"/>
@@
 <instance part="RST" gate="G$1" x="172.72" y="187.96" smashed="yes" rot="R270">
 <attribute name="NAME" x="177.8" y="181.61" size="1.778" layer="95" rot="R270" align="center-left"/>
+</instance>
+<instance part="C2" gate="G$1" x="88.9" y="198.12" smashed="yes">
+<attribute name="NAME" x="90.424" y="198.501" size="1.778" layer="95"/>
+<attribute name="VALUE" x="90.424" y="193.421" size="1.778" layer="96"/>
 </instance>
 </instances>
@@
 <wire x1="101.6" y1="182.88" x2="88.9" y2="182.88" width="0.1524" layer="91"/>
 <wire x1="88.9" y1="182.88" x2="88.9" y2="167.64" width="0.1524" layer="91"/>
-<pinref part="C2" gate="G$1" pin="2"/>
 <wire x1="88.9" y1="193.04" x2="88.9" y2="182.88" width="0.1524" layer="91"/>
 <junction x="88.9" y="182.88"/>
 <pinref part="GND2" gate="1" pin="GND"/>
+<pinref part="C2" gate="G$1" pin="2"/>
 </segment>
 <segment>
@@
 <wire x1="83.82" y1="203.2" x2="83.82" y2="210.82" width="0.1524" layer="91"/>
 <label x="83.82" y="210.82" size="1.778" layer="95" rot="R90" xref="yes"/>
-<pinref part="C2" gate="G$1" pin="1"/>
 <wire x1="88.9" y1="200.66" x2="88.9" y2="203.2" width="0.1524" layer="91"/>
 <junction x="88.9" y="203.2"/>
@@
 <wire x1="106.68" y1="198.12" x2="106.68" y2="203.2" width="0.1524" layer="91"/>
 <junction x="106.68" y="203.2"/>
-</segment>
-<segment>
+<pinref part="C2" gate="G$1" pin="1"/>
+</segment>
+<segment>

Commit message: numitron 4 resistor error correction
Connections:
- removed net IO15: SV1.6
- net GPIO15: now also SV1.6
Changed lines of the file:
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@@
 <label x="160.02" y="200.66" size="1.778" layer="95"/>
+</segment>
+<segment>
+<wire x1="238.76" y1="203.2" x2="248.92" y2="203.2" width="0.1524" layer="91"/>
+<label x="238.76" y="203.2" size="1.778" layer="95"/>
+<pinref part="SV1" gate="1" pin="6"/>
 </segment>
 </net>
@@
 <label x="238.76" y="165.1" size="1.778" layer="95"/>
 <pinref part="SV2" gate="1" pin="1"/>
-</segment>
-</net>
-<net name="IO15" class="0">
-<segment>
-<wire x1="238.76" y1="203.2" x2="248.92" y2="203.2" width="0.1524" layer="91"/>
-<label x="238.76" y="203.2" size="1.778" layer="95"/>
-<pinref part="SV1" gate="1" pin="6"/>
 </segment>
 </net>
@@
 </sheet>
 </sheets>
-<errors>
-</errors>
 </schematic>
 </drawing>
