File: designs/NixiTubeClock/3.3V_StepDown.sch (EAGLE design)
At the start: 10 parts, among them IC1 TPS62160DGKR, J1 S2B-PH-SM4, J2 S2B-PH-SM4

Commit message: started work on mainboard
Parts:
- removed J1, J2: S2B-PH-SM4, CommonParts:S2B-PH-SM4
Connections:
- net AGND: no longer J1.2, J2.2
- net IOUT: no longer J2.1
- net VIN: no longer J1.1
Changed lines of the file:
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@@
 <?xml version="1.0" encoding="utf-8"?>
 <!DOCTYPE eagle SYSTEM "eagle.dtd">
-<eagle version="9.4.2">
+<eagle version="9.5.1">
 <drawing>
 <settings>
@@
 <part name="AGND4" library="supply1" library_urn="urn:adsk.eagle:library:371" deviceset="AGND" device=""/>
 <part name="AGND5" library="supply1" library_urn="urn:adsk.eagle:library:371" deviceset="AGND" device=""/>
-<part name="J1" library="CommonParts" deviceset="S2B-PH-SM4" device=""/>
-<part name="J2" library="CommonParts" deviceset="S2B-PH-SM4" device=""/>
-<part name="AGND2" library="supply1" library_urn="urn:adsk.eagle:library:371" deviceset="AGND" device=""/>
-<part name="AGND3" library="supply1" library_urn="urn:adsk.eagle:library:371" deviceset="AGND" device=""/>
 <part name="L1" library="MouserUseful" deviceset="VLS6045EX-221M" device=""/>
 </parts>
@@
 <instance part="AGND5" gate="VR1" x="142.24" y="93.98" smashed="yes">
 <attribute name="VALUE" x="139.7" y="88.9" size="1.778" layer="96" rot="R90"/>
-</instance>
-<instance part="J1" gate="G$1" x="104.14" y="111.76" smashed="yes" rot="R90">
-<attribute name="NAME" x="98.54428125" y="106.6771" size="1.272509375" layer="95" rot="R90"/>
-<attribute name="VALUE" x="113.56268125" y="106.67188125" size="1.275409375" layer="96" rot="R90"/>
-</instance>
-<instance part="J2" gate="G$1" x="121.92" y="111.76" smashed="yes" rot="R90">
-<attribute name="NAME" x="116.32428125" y="106.6771" size="1.272509375" layer="95" rot="R90"/>
-<attribute name="VALUE" x="131.34268125" y="106.67188125" size="1.275409375" layer="96" rot="R90"/>
-</instance>
-<instance part="AGND2" gate="VR1" x="109.22" y="91.44" smashed="yes">
-<attribute name="VALUE" x="106.68" y="86.36" size="1.778" layer="96" rot="R90"/>
-</instance>
-<instance part="AGND3" gate="VR1" x="127" y="91.44" smashed="yes">
-<attribute name="VALUE" x="124.46" y="86.36" size="1.778" layer="96" rot="R90"/>
 </instance>
 <instance part="L1" gate="G$1" x="106.68" y="154.94" smashed="yes">
@@
 <wire x1="137.16" y1="111.76" x2="137.16" y2="106.68" width="0.1524" layer="91"/>
 <label x="137.16" y="106.68" size="1.778" layer="95" rot="R270" xref="yes"/>
-</segment>
-<segment>
-<pinref part="J1" gate="G$1" pin="1"/>
-<wire x1="101.6" y1="104.14" x2="101.6" y2="101.6" width="0.1524" layer="91"/>
-<label x="101.6" y="101.6" size="1.778" layer="95" rot="R270" xref="yes"/>
 </segment>
 </net>
@@
 <wire x1="144.78" y1="111.76" x2="144.78" y2="106.68" width="0.1524" layer="91"/>
 <label x="144.78" y="106.68" size="1.778" layer="95" rot="R270" xref="yes"/>
-</segment>
-<segment>
-<pinref part="J2" gate="G$1" pin="1"/>
-<wire x1="119.38" y1="104.14" x2="119.38" y2="101.6" width="0.1524" layer="91"/>
-<label x="119.38" y="101.6" size="1.778" layer="95" rot="R270" xref="yes"/>
 </segment>
 </net>
@@
 <wire x1="142.24" y1="96.52" x2="142.24" y2="111.76" width="0.1524" layer="91"/>
 </segment>
-<segment>
-<pinref part="J1" gate="G$1" pin="2"/>
-<wire x1="104.14" y1="104.14" x2="104.14" y2="93.98" width="0.1524" layer="91"/>
-<pinref part="AGND2" gate="VR1" pin="AGND"/>
-<wire x1="104.14" y1="93.98" x2="109.22" y2="93.98" width="0.1524" layer="91"/>
-</segment>
-<segment>
-<pinref part="J2" gate="G$1" pin="2"/>
-<pinref part="AGND3" gate="VR1" pin="AGND"/>
-<wire x1="121.92" y1="104.14" x2="121.92" y2="93.98" width="0.1524" layer="91"/>
-<wire x1="121.92" y1="93.98" x2="127" y2="93.98" width="0.1524" layer="91"/>
-</segment>
 </net>
