File: designs/NixiTubeClock/180V_StepUp.sch (EAGLE design)
At the start: 14 parts, among them IC1 MAX1771, Q1 RF644, X1 332-08

Commit message: started work on mainboard
Parts:
- removed X1: 332-08, con-garry:332-08
- added LED1: GREEN, CommonParts:LED_1206SMT1206
- added R4: 1K, CommonParts:R-EU_1206R1206
- added SV2: (no value), con-lstb:MA08-1
Connections:
- new net N$1: LED1.A, R4.2
- net +170V: now also SV2.7, SV2.8; no longer X1-8.S
- net GND: now also LED1.C, SV2.3, SV2.4, SV2.5, SV2.6; no longer X1-2.S, X1-3.S, X1-4.S, X1-5.S, X1-6.S, X1-7.S
- net VIN: now also R4.1, SV2.1, SV2.2; no longer X1-1.S
Other:
- note added: "Nothing just Picture"
