File: designs/NixiTubeClock/180V_StepUp.brd (EAGLE design)
At the start: 50 x 38 mm, 14 parts, among them IC1 MAX1771, Q1 RF644, X1 332-08

Commit message: added new nixi clock design top board
Parts:
- moved C1 2.00 mm to (20.9, 9.93)
- moved C2 2.00 mm to (21.4, 17.0)
- moved C3 2.00 mm to (39.8, 15.0)
- moved C4 2.00 mm to (46.4, 29.9)
- moved C5 2.00 mm to (45.4, 20.2)
- moved D1 2.00 mm to (33.0, 32.0)
- moved IC1 2.00 mm to (28.4, 15.6)
- moved L1 2.00 mm to (14.2, 31.1)
- moved Q1 2.00 mm to (28.0, 26.0)
- moved R1 2.00 mm to (37.1, 11.0)
- moved R2 2.00 mm to (32.9, 6.82)
- moved R3 2.00 mm to (44.1, 9.04)
- moved RS1 2.00 mm to (37.6, 22.9)
- moved X1 2.00 mm to (27.0, 2.00)
Other:
- board size 50 x 38 mm -> 54 x 40 mm

Commit message: started work on mainboard
Parts:
- removed X1: 332-08, con-garry:332-08
- added LED1: GREEN, CommonParts:1206
- added R4: 1K, CommonParts:R1206
- added SV2: (no value), con-lstb:MA08-1
- moved R2 1.80 mm to (31.9, 8.32)
- moved R1 1.41 mm to (36.1, 12.0)
- moved C1 1.00 mm to (19.9, 9.93)
- moved C2 1.00 mm to (20.4, 17.0)
- moved C3 1.00 mm to (38.8, 15.0)
- moved C4 1.00 mm to (45.4, 29.9)
- moved C5 1.00 mm to (44.4, 20.2)
- moved D1 1.00 mm to (32.0, 32.0)
- moved IC1 1.00 mm to (27.4, 15.6)
- moved L1 1.00 mm to (13.2, 31.1)
- moved Q1 1.00 mm to (27.0, 26.0)
- moved R3 1.00 mm to (43.1, 9.04)
- moved RS1 1.00 mm to (36.6, 22.9)
Connections:
- new net N$1: LED1.A, R4.2
- net +170V: now also SV2.7, SV2.8; no longer X1.8
- net GND: now also LED1.C, SV2.3, SV2.4, SV2.5, SV2.6; no longer X1.2, X1.3, X1.4, X1.5, X1.6, X1.7
- net VIN: now also R4.1, SV2.1, SV2.2; no longer X1.1
Routing:
- net VIN: track 78.2 -> 12.5 mm
- net N$1: track 0.00 -> 4.00 mm
- net +170V: track 3.41 -> 3.95 mm
- net GND: vias 16 -> 15
Other:
- board size 54 x 40 mm -> 52 x 39 mm
- board text added: "12-15V 170-220V"
- board text added: "12V"
- board text added: "170V"
- board text added: "GND"
- board text removed: "Vin 12 - 15"
- board text removed: "Vout 150 - 220"
- board text removed: "in"
- board text removed: "out"

Commit message: integrated T/H sensor
Parts:
- moved Q1 5.00 mm to (27.0, 21.0), flipped to the bottom, turned to 180 degrees
Routing:
- net VIN: track 12.5 -> 15.0 mm
Other:
- board text added: "HIGH VOLTAGE"

Commit message: added new cam data and made last checks before order :o
Routing:
- net GND: track 37.7 -> 38.3 mm
Changed lines of the file:
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@@
 <drawing>
 <settings>
-<setting alwaysvectorfont="yes"/>
+<setting alwaysvectorfont="no"/>
 <setting verticaltext="up"/>
 </settings>
@@
 </layers>
 <board>
-<fusionsync huburn="a.cGVyc29uYWw6dWUyYTNmMDU1" projecturn="a.cGVyc29uYWw6dWUyYTNmMDU1IzIwMTgxMjEwMTY0OTQ5MjI2" f3durn="urn:adsk.wipprod:dm.lineage:EW_nxjs3TOeM8ciUlo7Bhg" pcbguid="f30d4857-b7eb-4cd6-9f83-62fb7e7f0654" lastpulledtime="" lastsyncedchangeguid="197d38ea-c724-6cd4-b45d-e32d125fc2c5"/>
+<fusionsync huburn="a.cGVyc29uYWw6dWUyYTNmMDU1" projecturn="a.cGVyc29uYWw6dWUyYTNmMDU1IzIwMTgxMjEwMTY0OTQ5MjI2" f3durn="urn:adsk.wipprod:dm.lineage:EW_nxjs3TOeM8ciUlo7Bhg" pcbguid="f30d4857-b7eb-4cd6-9f83-62fb7e7f0654" lastpulledtime="" lastsyncedchangeguid="e5bd292d-e348-6bac-0a30-bca2dcfeea96"/>
 <plain>
 <wire x1="51" y1="2" x2="51" y2="37" width="0" layer="20"/>
@@
 <hole x="2" y="36" drill="2.8"/>
 <hole x="48" y="36" drill="2.8"/>
-<text x="15.5" y="4" size="1.016" layer="26" rot="R90">12V</text>
-<text x="18.057140625" y="4" size="1.016" layer="26" rot="R90">12V</text>
-<text x="20.61428125" y="4" size="1.016" layer="26" rot="R90">GND</text>
-<text x="23.171421875" y="4" size="1.016" layer="26" rot="R90">GND</text>
-<text x="25.7285625" y="4" size="1.016" layer="26" rot="R90">GND</text>
-<text x="28.285703125" y="4" size="1.016" layer="26" rot="R90">GND</text>
-<text x="30.84284375" y="4" size="1.016" layer="26" rot="R90">170V</text>
-<text x="33.399984375" y="4" size="1.016" layer="26" rot="R90">170V</text>
+<text x="37.5" y="1" size="1.016" layer="25" rot="R90">12V</text>
+<text x="39.057140625" y="1" size="1.016" layer="25" rot="R90">12V</text>
+<text x="40.61428125" y="1" size="1.016" layer="25" rot="R90">GND</text>
+<text x="42.171421875" y="1" size="1.016" layer="25" rot="R90">GND</text>
+<text x="43.7285625" y="1" size="1.016" layer="25" rot="R90">GND</text>
+<text x="45.285703125" y="1" size="1.016" layer="25" rot="R90">GND</text>
+<text x="46.84284375" y="1" size="1.016" layer="25" rot="R90">170V</text>
+<text x="48.399984375" y="1" size="1.016" layer="25" rot="R90">170V</text>
 <text x="5.5" y="4.2" size="1.016" layer="25" ratio="10" distance="10" rot="R90">12-15V 170-220V</text>
 <dimension x1="2" y1="36" x2="48" y2="36" x3="25" y3="41" textsize="1.778" layer="47" dtype="horizontal"/>
@@
 </class>
 </classes>
-<designrules name="default">
+<designrules name="default *">
 <description language="de">&lt;b&gt;EAGLE Design Rules&lt;/b&gt;
 &lt;p&gt;
@@
 <param name="mdViaViaSameLayer" value="6mil"/>
 <param name="mnLayersViaInSmd" value="2"/>
-<param name="mdCopperDimension" value="40mil"/>
+<param name="mdCopperDimension" value="10mil"/>
 <param name="mdDrill" value="6mil"/>
 <param name="mdSmdStop" value="0mil"/>
@@
 <via x="42.7" y="10.3" extent="1-16" drill="0.1"/>
 <polygon width="0" layer="16">
-<vertex x="50" y="36"/>
-<vertex x="50" y="2" curve="-90"/>
-<vertex x="48" y="0"/>
-<vertex x="2" y="0" curve="-90"/>
-<vertex x="0" y="2"/>
-<vertex x="0" y="36" curve="-90"/>
-<vertex x="2" y="38"/>
-<vertex x="48" y="38" curve="-90"/>
+<vertex x="51" y="38"/>
+<vertex x="51" y="0"/>
+<vertex x="0" y="0" curve="-90"/>
+<vertex x="-1" y="1"/>
+<vertex x="-1" y="37" curve="-90"/>
+<vertex x="1" y="39"/>
+<vertex x="50" y="39" curve="-90"/>
 </polygon>
 <polygon width="0" layer="16">
-<vertex x="50" y="36"/>
-<vertex x="50" y="2" curve="-90"/>
-<vertex x="48" y="0"/>
-<vertex x="2" y="0" curve="-90"/>
-<vertex x="0" y="2"/>
-<vertex x="0" y="36" curve="-90"/>
-<vertex x="2" y="38"/>
-<vertex x="48" y="38" curve="-90"/>
+<vertex x="50.95" y="37.05"/>
+<vertex x="50.95" y="1.95" curve="-90"/>
+<vertex x="49" y="0"/>
+<vertex x="1" y="0" curve="-90"/>
+<vertex x="-1" y="2"/>
+<vertex x="-1" y="37" curve="-90"/>
+<vertex x="1" y="39"/>
+<vertex x="49" y="39" curve="-90"/>
 </polygon>
 <contactref element="SV2" pad="3"/>
@@
 <contactref element="SV2" pad="6"/>
 <contactref element="LED1" pad="C"/>
-<wire x1="43.5" y1="9.7" x2="43.13" y2="9.99" width="0" layer="19" extent="1-1"/>
+<wire x1="43.13" y1="9.99" x2="43.01" y2="9.99" width="0.1524" layer="1"/>
+<wire x1="43.01" y1="9.99" x2="42.7" y2="10.3" width="0.1524" layer="1"/>
 </signal>
 <signal name="N$2">
@@
 <contactref element="R1" pad="2"/>
 <polygon width="0.1524" layer="1">
-<vertex x="51" y="9.3"/>
-<vertex x="37" y="9.3"/>
+<vertex x="51" y="9.4"/>
+<vertex x="37" y="9.4"/>
 <vertex x="37" y="13"/>
 <vertex x="40.5" y="13"/>
@@
 <mfgpreviewcolor name="substratecolor" color="0xFF786E46"/>
 </mfgpreviewcolors>
+<errors>
+</errors>
 </board>
 </drawing>
