File: designs/EasterRadio/power.sch (EAGLE design)
At the start: 13 parts, among them IC1 MCP73832T-2ACI_OT, IC3 DMP1045U-7, J4 S2B-PH-SM4, J6 PJ-002AH-SMT-TR

Commit message: changed to correct diode and designed power pcb
Parts:
- D1: value 1N4942 -> LSM115JE3_TR13; device diode:1N4942 -> CommonParts:LSM115JE3_TR13
Connections:
- removed net 12V: C30.1, D1.C, IC3.D, J6.1_1, J6.1_2, JP1.1
- new net U_DRAIN: C30.1, D1.K, IC3.D, JP1.1
- net 5V: now also J6.1_1, J6.1_2
- net GNDA: no longer J4.SHIELD
Other:
- note removed: "Power"
Changed lines of the file:
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@@
 <setting verticaltext="up"/>
 </settings>
-<grid distance="0.1" unitdist="inch" unit="inch" style="lines" multiple="1" display="no" altdistance="0.01" altunitdist="inch" altunit="inch"/>
+<grid distance="0.05" unitdist="inch" unit="inch" style="lines" multiple="1" display="yes" altdistance="0.01" altunitdist="inch" altunit="inch"/>
 <layers>
 <layer number="1" name="Top" color="4" fill="1" visible="no" active="no"/>
@@
 </variantdefs>
 <classes>
-<class number="0" name="default" width="0" drill="0">
+<class number="0" name="default" width="0.7" drill="0.8">
+<clearance class="0" value="0.2"/>
 </class>
 </classes>
@@
 <part name="JP1" library="pinhead" library_urn="urn:adsk.eagle:library:325" deviceset="PINHD-1X4" device="" package3d_urn="urn:adsk.eagle:package:22407/2"/>
 <part name="IC3" library="MouserUseful" deviceset="DMP1045U-7" device=""/>
-<part name="D1" library="diode" library_urn="urn:adsk.eagle:library:210" deviceset="1N4942" device="" package3d_urn="urn:adsk.eagle:package:43336/1"/>
 <part name="R14" library="CommonParts" deviceset="R-EU_1206" device="R1206" package3d_urn="urn:adsk.eagle:package:23540/2" value="100K"/>
 <part name="GND9" library="supply1" library_urn="urn:adsk.eagle:library:371" deviceset="GNDA" device=""/>
 <part name="C30" library="CommonParts" deviceset="C-EU_805" device="C0805" package3d_urn="urn:adsk.eagle:package:23617/2" value="1uF"/>
+<part name="D1" library="CommonParts" deviceset="LSM115JE3_TR13" device=""/>
 </parts>
 <sheets>
@@
 <text x="0" y="120.65" size="5.08" layer="91">Power
 (MCP73832T-2ACI/OT)</text>
-<text x="151.13" y="109.22" size="2.54" layer="91">Power</text>
 <frame x1="0" y1="0" x2="186.69" y2="118.11" columns="8" rows="5" layer="91"/>
 <text x="149.86" y="78.74" size="1.778" layer="91">Step down to 3.3V Converter</text>
@@
 <attribute name="VALUE" x="125.73" y="49.53" size="1.778" layer="96" align="center-left"/>
 </instance>
-<instance part="D1" gate="1" x="144.78" y="54.61" smashed="yes" rot="R270">
-<attribute name="NAME" x="145.2626" y="52.07" size="1.778" layer="95" rot="R270"/>
-<attribute name="VALUE" x="142.4686" y="52.07" size="1.778" layer="96" rot="R270"/>
-</instance>
 <instance part="R14" gate="G$1" x="157.48" y="55.88" smashed="yes" rot="R270">
 <attribute name="NAME" x="161.5186" y="53.34" size="1.778" layer="95" rot="R90"/>
@@
 <attribute name="NAME" x="146.304" y="32.131" size="1.778" layer="95"/>
 <attribute name="VALUE" x="146.304" y="27.051" size="1.778" layer="96"/>
+</instance>
+<instance part="D1" gate="G$1" x="144.78" y="43.18" smashed="yes" rot="R90">
+<attribute name="NAME" x="135.89" y="55.88" size="1.778" layer="95" rot="R90" align="center-left"/>
+<attribute name="VALUE" x="138.43" y="55.88" size="1.778" layer="96" rot="R90" align="center-left"/>
 </instance>
 </instances>
@@
 <wire x1="82.55" y1="40.64" x2="77.47" y2="40.64" width="0.1524" layer="91"/>
 <wire x1="77.47" y1="40.64" x2="77.47" y2="35.56" width="0.1524" layer="91"/>
-<pinref part="J4" gate="G$1" pin="SHIELD"/>
-<wire x1="82.55" y1="35.56" x2="77.47" y2="35.56" width="0.1524" layer="91"/>
 <junction x="77.47" y="35.56"/>
 <pinref part="C26" gate="G$1" pin="1"/>
@@
 </segment>
 </net>
-<net name="12V" class="0">
-<segment>
-<pinref part="J6" gate="G$1" pin="1_2"/>
-<wire x1="95.25" y1="82.55" x2="99.06" y2="82.55" width="0.1524" layer="91"/>
-<pinref part="J6" gate="G$1" pin="1_1"/>
-<wire x1="95.25" y1="80.01" x2="99.06" y2="80.01" width="0.1524" layer="91"/>
-<wire x1="99.06" y1="82.55" x2="99.06" y2="80.01" width="0.1524" layer="91"/>
-<wire x1="99.06" y1="82.55" x2="99.06" y2="87.63" width="0.1524" layer="91"/>
-<junction x="99.06" y="82.55"/>
-</segment>
-<segment>
-<pinref part="JP1" gate="A" pin="1"/>
-<pinref part="IC3" gate="G$1" pin="D"/>
-<wire x1="129.54" y1="44.45" x2="144.78" y2="44.45" width="0.1524" layer="91"/>
-<pinref part="D1" gate="1" pin="C"/>
-<wire x1="144.78" y1="44.45" x2="144.78" y2="52.07" width="0.1524" layer="91"/>
-<wire x1="144.78" y1="44.45" x2="144.78" y2="34.29" width="0.1524" layer="91"/>
-<junction x="144.78" y="44.45"/>
-<wire x1="170.18" y1="73.66" x2="170.18" y2="44.45" width="0.1524" layer="91"/>
-<wire x1="170.18" y1="44.45" x2="144.78" y2="44.45" width="0.1524" layer="91"/>
-<pinref part="C30" gate="G$1" pin="1"/>
-</segment>
-</net>
 <net name="5V" class="0">
 <segment>
@@
 <wire x1="109.22" y1="44.45" x2="109.22" y2="62.23" width="0.1524" layer="91"/>
 <wire x1="109.22" y1="62.23" x2="144.78" y2="62.23" width="0.1524" layer="91"/>
-<wire x1="144.78" y1="62.23" x2="144.78" y2="57.15" width="0.1524" layer="91"/>
-<pinref part="D1" gate="1" pin="A"/>
+<pinref part="R14" gate="G$1" pin="1"/>
 <wire x1="144.78" y1="62.23" x2="157.48" y2="62.23" width="0.1524" layer="91"/>
-<junction x="144.78" y="62.23"/>
-<pinref part="R14" gate="G$1" pin="1"/>
 <wire x1="157.48" y1="62.23" x2="157.48" y2="60.96" width="0.1524" layer="91"/>
 <pinref part="LED2" gate="G$1" pin="A"/>
@@
 <junction x="17.78" y="38.1"/>
 <junction x="109.22" y="62.23"/>
+<pinref part="D1" gate="G$1" pin="A"/>
+<wire x1="144.78" y1="60.96" x2="144.78" y2="62.23" width="0.1524" layer="91"/>
+<junction x="144.78" y="62.23"/>
 </segment>
 <segment>
 <label x="99.06" y="87.63" size="1.778" layer="95" rot="R90" xref="yes"/>
+</segment>
+<segment>
+<pinref part="J6" gate="G$1" pin="1_2"/>
+<wire x1="95.25" y1="82.55" x2="99.06" y2="82.55" width="0.1524" layer="91"/>
+<pinref part="J6" gate="G$1" pin="1_1"/>
+<wire x1="95.25" y1="80.01" x2="99.06" y2="80.01" width="0.1524" layer="91"/>
+<wire x1="99.06" y1="82.55" x2="99.06" y2="80.01" width="0.1524" layer="91"/>
+<wire x1="99.06" y1="82.55" x2="99.06" y2="87.63" width="0.1524" layer="91"/>
+<junction x="99.06" y="82.55"/>
 </segment>
 </net>
@@
 <label x="177.8" y="53.34" size="1.778" layer="95" rot="R270" xref="yes"/>
 </segment>
-<segment>
-<wire x1="151.13" y1="104.14" x2="161.29" y2="104.14" width="0.1524" layer="91"/>
-<label x="161.29" y="104.14" size="1.778" layer="95" xref="yes"/>
-</segment>
-</net>
-<net name="AGND" class="0">
-<segment>
-<wire x1="151.13" y1="99.06" x2="161.29" y2="99.06" width="0.1524" layer="91"/>
-<label x="161.29" y="99.06" size="1.778" layer="95" xref="yes"/>
-</segment>
-</net>
+</net>
+<net name="U_DRAIN" class="0">
+<segment>
+<pinref part="JP1" gate="A" pin="1"/>
+<pinref part="IC3" gate="G$1" pin="D"/>
+<wire x1="170.18" y1="73.66" x2="170.18" y2="44.45" width="0.1524" layer="91"/>
+<wire x1="170.18" y1="44.45" x2="144.78" y2="44.45" width="0.1524" layer="91"/>
+<pinref part="D1" gate="G$1" pin="K"/>
+<wire x1="144.78" y1="44.45" x2="129.54" y2="44.45" width="0.1524" layer="91"/>
+<wire x1="144.78" y1="45.72" x2="144.78" y2="44.45" width="0.1524" layer="91"/>
+<junction x="144.78" y="44.45"/>
+<pinref part="C30" gate="G$1" pin="1"/>
+<wire x1="144.78" y1="44.45" x2="144.78" y2="34.29" width="0.1524" layer="91"/>
+</segment>
+</net>
