File: designs/TubeClock/MainBoard/MainBoard.brd (EAGLE design)
At the start: 98 x 67 mm, 46 parts, among them IC1 LD117ADT-TR, J1 S2B-NSHSS-TB, J2 S2B-NSHSS-TB, J3 S2B-NSHSS-TB, J4 PJ-002AH-SMT-TR, J5 S2B-NSHSS-TB, Q1 2N7002NXAKR, Q2 2N7002NXAKR

Commit message: small changes to easter radio mainboard started for in14 nixi tubes and cleanup
Parts:
- removed ALARM: F/QMBIII, buzzer:F/QMBIII
Connections:
- net GND: no longer ALARM.+
- net IO18: no longer ALARM.-
Routing:
- net GND: track 332.1 -> 292.2 mm
- net IO18: track 49.7 -> 44.0 mm
Changed lines of the file:
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@@
 <?xml version="1.0" encoding="utf-8"?>
 <!DOCTYPE eagle SYSTEM "eagle.dtd">
-<eagle version="9.5.1">
+<eagle version="9.6.2">
 <drawing>
 <settings>
@@
 <layer number="14" name="Route14" color="22" fill="1" visible="no" active="no"/>
 <layer number="15" name="Route15" color="23" fill="1" visible="no" active="no"/>
-<layer number="16" name="Bottom" color="1" fill="1" visible="no" active="yes"/>
+<layer number="16" name="Bottom" color="1" fill="1" visible="yes" active="yes"/>
 <layer number="17" name="Pads" color="2" fill="1" visible="yes" active="yes"/>
 <layer number="18" name="Vias" color="2" fill="1" visible="yes" active="yes"/>
@@
 </layers>
 <board>
-<fusionsync huburn="a.cGVyc29uYWw6dWUyYTNmMDU1" projecturn="a.cGVyc29uYWw6dWUyYTNmMDU1IzIwMTgxMjEwMTY0OTQ5MjI2" f3durn="urn:adsk.wipprod:dm.lineage:sIc1WYWiRnKTMBUjB1WWbw" pcbguid="963d08c0-42bd-4bef-8ac7-da9e1254c3c3" lastpulledtime="" lastsyncedchangeguid="7b91f2f7-91e4-476c-4a86-15bcad2ed177"/>
+<fusionsync huburn="a.cGVyc29uYWw6dWUyYTNmMDU1" projecturn="a.cGVyc29uYWw6dWUyYTNmMDU1IzIwMTgxMjEwMTY0OTQ5MjI2" f3durn="urn:adsk.wipprod:dm.lineage:sIc1WYWiRnKTMBUjB1WWbw" pcbguid="963d08c0-42bd-4bef-8ac7-da9e1254c3c3" lastpulledtime="" lastsyncedchangeguid="7b91f2f7-91e4-476c-4a86-15bcad2ed177" latestrevisionid="" lastsyncedrevisionid="" lastboardhashguid="" lastpushedtime="" linktopcb3d="false"/>
 <plain>
 <hole x="3" y="50" drill="2.8"/>
@@
 <attribute name="VALUE" x="37.38" y="6.075" size="1.27" layer="27" rot="R180"/>
 </element>
-<element name="ALARM" library="buzzer" library_urn="urn:adsk.eagle:library:113" package="F/QMBIII" package3d_urn="urn:adsk.eagle:package:5267/1" value="F/QMBIII" x="12" y="46" smashed="yes" rot="R180">
-<attribute name="MF" value="" x="12" y="46" size="1.778" layer="27" rot="R180" display="off"/>
-<attribute name="MPN" value="" x="12" y="46" size="1.778" layer="27" rot="R180" display="off"/>
-<attribute name="NAME" x="4.055" y="46.055" size="1.27" layer="25" ratio="10" rot="R270"/>
-<attribute name="OC_FARNELL" value="unknown" x="12" y="46" size="1.778" layer="27" rot="R180" display="off"/>
-<attribute name="OC_NEWARK" value="unknown" x="12" y="46" size="1.778" layer="27" rot="R180" display="off"/>
-<attribute name="POPULARITY" value="1" x="12" y="46" size="1.778" layer="27" rot="R180" display="off"/>
-</element>
 </elements>
 <signals>
@@
 <contactref element="Q2" pad="2"/>
 <contactref element="Q1" pad="2"/>
-<wire x1="8.7488" y1="50.66" x2="29.5" y2="50.66" width="0.8128" layer="16"/>
 <wire x1="11.73" y1="32.8" x2="14.27" y2="32.8" width="0.8128" layer="16"/>
 <wire x1="3.25" y1="12.25" x2="11.73" y2="12.25" width="0.8128" layer="16"/>
@@
 <wire x1="34.5" y1="48" x2="53" y2="48" width="0.6096" layer="1"/>
 <wire x1="56.8932" y1="49.3932" x2="59" y2="51.5" width="0.6096" layer="1"/>
-<contactref element="ALARM" pad="+"/>
-<wire x1="8.7488" y1="50.66" x2="8.7488" y2="46" width="0.8128" layer="16"/>
-<wire x1="11.73" y1="32.8" x2="11.73" y2="36.0188" width="0.8128" layer="16"/>
-<wire x1="11.73" y1="36.0188" x2="8.7488" y2="39" width="0.8128" layer="16"/>
-<wire x1="8.7488" y1="39" x2="8.7488" y2="46" width="0.8128" layer="16"/>
 <contactref element="J4" pad="3"/>
 <contactref element="J4" pad="4"/>
@@
 <wire x1="84" y1="5" x2="86.25" y2="7.25" width="0.2032" layer="1"/>
 <wire x1="86.25" y1="7.25" x2="86.25" y2="8.25" width="0.2032" layer="1"/>
-<wire x1="70.8" y1="8.6" x2="70.5" y2="7" width="0" layer="19" extent="1-16"/>
 </signal>
 <signal name="3.3V">
@@
 <signal name="IO18">
 <contactref element="SV5" pad="8"/>
-<contactref element="ALARM" pad="-"/>
-<wire x1="15.2512" y1="46" x2="15.2512" y2="40.2512" width="0.6096" layer="16"/>
 <wire x1="15.2512" y1="40.2512" x2="15" y2="40" width="0.8128" layer="16"/>
 <via x="15" y="40" extent="1-16" drill="0.8"/>
