File: designs/TubeClock/MainBoard/MainBoard.sch (EAGLE design)
At the start: 46 parts, among them IC1 LD117ADT-TR, J1 S2B-NSHSS-TB, J2 S2B-NSHSS-TB, J3 S2B-NSHSS-TB, J4 PJ-002AH-SMT-TR, J5 S2B-NSHSS-TB, Q1 2N7002NXAKR, Q2 2N7002NXAKR

Commit message: small changes to easter radio mainboard started for in14 nixi tubes and cleanup
Parts:
- removed ALARM: F/QMBIII, buzzer:F/QMBIII
Connections:
- net GND: no longer ALARM.-
- net IO18: no longer ALARM.+
Changed lines of the file:
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@@
 <?xml version="1.0" encoding="utf-8"?>
 <!DOCTYPE eagle SYSTEM "eagle.dtd">
-<eagle version="9.5.1">
+<eagle version="9.6.2">
 <drawing>
 <settings>
@@
 <part name="C4" library="CommonParts" deviceset="C-EU_805" device="C0805" package3d_urn="urn:adsk.eagle:package:23617/2" value="20nF"/>
 <part name="JP2" library="pinhead" library_urn="urn:adsk.eagle:library:325" deviceset="PINHD-1X4" device="" package3d_urn="urn:adsk.eagle:package:22407/2"/>
-<part name="ALARM" library="buzzer" library_urn="urn:adsk.eagle:library:113" deviceset="F/QMBIII" device="" package3d_urn="urn:adsk.eagle:package:5267/1"/>
-<part name="GND12" library="supply1" library_urn="urn:adsk.eagle:library:371" deviceset="GND" device=""/>
 <part name="GND11" library="supply1" library_urn="urn:adsk.eagle:library:371" deviceset="GND" device=""/>
 </parts>
@@
 <attribute name="VALUE" x="106.68" y="166.37" size="1.778" layer="96" rot="R90"/>
 </instance>
-<instance part="ALARM" gate="G$1" x="99.06" y="33.02" smashed="yes" rot="R270">
-<attribute name="NAME" x="105.41" y="35.56" size="1.778" layer="95" rot="R270"/>
-<attribute name="VALUE" x="99.06" y="27.94" size="1.778" layer="96" rot="R270"/>
-</instance>
-<instance part="GND12" gate="1" x="96.52" y="15.24" smashed="yes">
-<attribute name="VALUE" x="93.98" y="12.7" size="1.778" layer="96"/>
-</instance>
 <instance part="GND11" gate="1" x="76.2" y="66.04" smashed="yes">
 <attribute name="VALUE" x="73.66" y="63.5" size="1.778" layer="96"/>
@@
 </segment>
 <segment>
-<pinref part="GND12" gate="1" pin="GND"/>
-<pinref part="ALARM" gate="G$1" pin="-"/>
-<wire x1="96.52" y1="27.94" x2="96.52" y2="17.78" width="0.1524" layer="91"/>
-</segment>
-<segment>
 <pinref part="J4" gate="G$1" pin="2"/>
 <pinref part="GND11" gate="1" pin="GND"/>
@@
 <pinref part="SV5" gate="1" pin="8"/>
 </segment>
-<segment>
-<pinref part="ALARM" gate="G$1" pin="+"/>
-<wire x1="96.52" y1="35.56" x2="96.52" y2="40.64" width="0.1524" layer="91"/>
-<label x="96.52" y="40.64" size="1.778" layer="95" rot="R90" xref="yes"/>
-</segment>
-</net>
+</net>

Commit message: changed mainboard design radio
Parts:
- removed SV2, SV3, SV4, SV5: (no value), CommonParts:PINHEADER-1X9
- added JP3, JP4: (no value), pinhead:PINHD-1X14
Connections:
- removed net CLK: SV4.9
- removed net CMD: SV3.1
- removed net EN: SV2.7
- removed net GPIO12: SV3.5
- removed net GPIO13: SV3.4
- removed net GPIO14: SV3.6
- removed net IO0: SV4.4
- removed net IO15: C3.1, J1.2, R1.2, SV4.6
- removed net IO18: SV5.8
- removed net IO19: SV5.7
- removed net IO2: SV1.3, SV4.5
- removed net IO23: SV5.1
- removed net IO4: SV1.1, SV4.3
- removed net IO5: SV1.2, SV5.9
- removed net NC_1: SV4.2
- removed net NC_2: SV4.1
- removed net NC_3: SV5.6
- removed net SD0: SV4.8
- removed net SD1: SV4.7
- removed net SD2: SV3.3
- removed net SD3: SV3.2
- removed net SEN_VN: SV2.5
- removed net SEN_VP: SV2.6
- new net IO12: C4.1, J3.2, JP3.13, R2.2
- new net IO13: C3.1, J1.2, JP3.14, R1.2
- new net IO14: JP3.12, R3.1
- new net SENSOR_VN: JP3.4
- new net SENSOR_VP: JP3.3
- net 3.3V: now also JP3.2; no longer SV2.8
- net GND: now also JP3.1, JP4.12, JP4.13, JP4.14; no longer SV2.9
- net IO21: now also JP4.8; no longer SV5.5
- net IO22: now also JP4.11; no longer SV5.2
- net IO25: now also JP3.9, SV1.2; no longer SV3.9
- net IO26: now also JP3.10, SV1.3; no longer R3.1, SV3.8
- net IO27: now also JP3.11; no longer SV3.7
- net IO32: now also JP3.7; no longer SV2.2
- net IO33: now also JP3.8, SV1.1; no longer SV2.1
- net IO34: now also JP3.5; no longer SV2.4
- net IO35: now also JP3.6; no longer SV2.3
- net RXD0: now also JP4.9; no longer C4.1, J3.2, R2.2, SV5.4
- net TXD0: now also JP4.10; no longer SV5.3
Other:
- note added: "Btn"
- note added: "LEDs"
- note removed: "IO03 Rx0"
